File: InterfaceBoard/dedica interface board.brd (EAGLE design)
At the start: 87.6 x 85.1 mm, 12 parts, among them J1 1x10 HEADER "A", J2 1x10 HEADER "B", J3 1x10 HEADER "C", J4 1x10 HEADER "D"

Commit message: Add SSR and Meanwell Libraries Add SSR and Power Supply to schematic
Parts:
- removed C2: 0.1uF, adafruit:C0603
- added C3: 100nf, OPL_Capacitor:C0603
- added D1, D2, D3: GREEN-0805, OPL_Optoelectronics:LED-0805
- added J10, J11, J9: GREEN-3P-5.0, OPL_Connector:H3-5.0-15.5X8.0MM
- added J12, J7, J8: (no value), SparkFun-Connectors:1X03
- added J13: (no value), SparkFun-Connectors:1X02
- added J6: (no value), SparkFun-Connectors:1X08
- added R10: 10K 1/10W, OPL_Resistor:R0603
- added R11, R12: 1.5K, OPL_Resistor:R0603
- added R6, R7, R8: DNP, adafruit:R0603
- added R9: TBC, adafruit:R0603
- added U$1: (no value), meanwell_irm_v7:IRM_01/02
- added U$2: AQ3A2-ZT4/32VDC, PanasonicAQ1:AQ3A2-ZT4/32VDC
- added U$3: AQ10A2-ZT4/32VDC, PanasonicAQ1:AQ10A2-ZT4/32VDC
- R1: value 4.7K -> 1K 1/10W; device adafruit:R0603 -> OPL_Resistor:R0603
- R2: value 10K -> 4.7K; device adafruit:R0603 -> OPL_Resistor:R0603
- R3: value 1K -> 4.7K; device adafruit:R0603 -> OPL_Resistor:R0603
- R4: device adafruit:R0603 -> OPL_Resistor:R0603
- R5: value 4.7K -> 1.5K; device adafruit:R0603 -> OPL_Resistor:R0603
- moved R5 166.4 mm to (-85.1, -215.9)
- moved R1 106.8 mm to (-64.8, -128.3)
- moved R3 98.8 mm to (-74.9, -128.3)
- moved R4 98.0 mm to (-80.0, -128.3)
- moved R2 97.6 mm to (-59.7, -128.3)
- flipped J1 to the bottom
Connections:
- new net 230VL: J9.1, U$1.AC/L, U$2.P$1, U$3.P$1
- new net 230VN: J10.1, J10.2, J10.3, J9.2, U$1.AC/N
- new net GND: J9.3
- new net HEATER_230VL: J11.1, U$3.P$2
- new net N$2: J6.2, J6.4, J6.6, J6.8
- new net N$3: D1.+, R11.2
- new net N$4: D3.+, R5.1
- new net N$5: D2.+, R12.1
- new net NTC_1: J6.1, R9.2
- new net NTC_2: J6.3, R8.2
- new net NTC_3: J6.5, R7.2
- new net NTC_4: J6.7, R6.2
- new net PGAUGE_1: J7.2
- new net PGAUGE_2: J8.2
- new net PUMP_230VL: J11.2, U$2.P$2
- new net RES_LCD_CLK: J1.7
- new net RES_LCD_CS: J1.6
- new net RES_LCD_DISP: J1.5
- new net RES_LCD_EXTCOMIN: J2.2
- new net RES_LCD_POWER: J1.2
- new net RES_MISO: J2.7
- new net RES_MOSI: J2.6
- new net RES_SD_CS: J1.8
- new net RES_SD_DET: J2.4
- net +5V: now also J12.1, J3.1, J7.1, J8.1, R10.2, R11.1, U$1.V+; no longer R1.2
- net AGND: now also C3.1, D1.-, D2.-, D3.-, J12.3, J13.2, J2.1, J3.2, J7.3, J8.3, R3.1, R6.1, R7.1, R8.1, R9.1, U$1.V-, U$2.P$4, U$3.P$4; no longer C2.2, R5.1
- net FLOW_SIG: now also J12.2, R2.1; no longer R1.1
- net HEATERSSR_CTRL: now also R12.2, R4.2, U$3.P$3; no longer R5.2
- net N$1: now also J13.1, R1.1; no longer R3.2
- net PUMPSSR_CTRL: now also R3.2, R5.2, U$2.P$3; no longer R4.2
- net STEAM_SW: now also C3.2, R1.2, R10.1; no longer C2.1, R2.1, R3.1

Commit message: 3.3V MCU updates
Parts:
- removed R3, R4: 4.7K, OPL_Resistor:R0603
- added C2, C4: 100nf, OPL_Capacitor:C0603
- added D4: GREEN-0805, OPL_Optoelectronics:LED-0805
- added J14: (no value), SparkFun-Connectors:1X06_LOCK
- added Q1, Q2: BSS138W-7-F, OPL_Discrete_Semiconductor:SOT-23
- added R13, R14: 1K 1/10W, OPL_Resistor:R0603
- added R15, R16: 1K, OPL_Resistor:R0805
- added R17: 1.5K, OPL_Resistor:R0603
- added R18, R19: 12K, OPL_Resistor:R0603
- added R20, R21: 30K, OPL_Resistor:R0603
- added R22, R23: 10K 1/10W, OPL_Resistor:R0603
- added R24, R25: 4.7K, OPL_Resistor:R0603
- C1: value 100nF -> 100nf; device adafruit:C0603 -> OPL_Capacitor:C0603
- moved U$3 240.4 mm to (63.5, 38.1), turned to 180 degrees
- moved C1 221.6 mm to (-130.8, -226.1)
- moved U$2 220.0 mm to (69.8, 15.2), turned to 270 degrees
- moved U$1 187.6 mm to (11.4, 29.2), turned to 270 degrees
- moved J11 182.9 mm to (34.3, 49.5), turned to 270 degrees
- moved J9 167.2 mm to (5.08, 50.8), turned to 270 degrees
Connections:
- removed net N$2: J6.2, J6.4, J6.6, J6.8
- new net 3.3V: J1.1, R10.2, R17.1, R2.2
- new net EXT_DR1: J14.2
- new net EXT_DR2: J14.1
- new net EXT_LED3: R16.2
- new net EXT_LED4: R15.2
- new net EXT_SW5: C2.2, R14.2
- new net EXT_SW6: C4.2, R13.2
- new net HEADERSSR_CTRL: J4.2
- new net N$10: J14.4, R15.1
- new net N$11: J14.3, R16.1
- new net N$14: Q2.2, R12.2, R23.1, U$3.P$3
- new net N$6: J14.6, R13.1
- new net N$7: J14.5, R14.1
- new net N$8: D4.+, R17.2
- new net PRES_1: J3.7, R18.1, R21.2
- new net PRES_2: J3.8, R19.1, R20.2
- new net W2: Q1.2, R22.1, R5.2, U$2.P$3
- net +5V: now also J6.2, J6.4, J6.6, J6.8, R22.2, R23.2; no longer R10.2, R2.2
- net AGND: now also C1.1, C2.1, C4.1, D4.-, Q1.3, Q2.3, R20.1, R21.1, R24.1, R25.1; no longer C1.2, R3.1, R4.1
- net FLOW_SIG: now also C1.2, J4.4; no longer C1.1
- net HEATERSSR_CTRL: now also Q2.1, R25.2; no longer R12.2, R4.2, U$3.P$3
- net NTC_1: now also J3.3
- net NTC_2: now also J3.4
- net NTC_3: now also J3.5
- net NTC_4: now also J3.6
- net PGAUGE_1: now also R18.2
- net PGAUGE_2: now also R19.2
- net PUMPSSR_CTRL: now also J4.1, Q1.1, R24.2; no longer R3.2, R5.2, U$2.P$3
- net STEAM_SW: now also J4.3
